Commit message: v1.1 stable gripper architecture + calibration + gazebo gui

File: my_robot_description/urdf/gripper_rg6.xacro (robot description, xacro)
@@ -142,4 +142,16 @@
     </collision>
   </link>
+  <link name="left_finger_contact_link"/>
+  <link name="right_finger_contact_link"/>
+  <joint name="left_finger_contact_joint" type="fixed">
+    <parent link="left_finger_tip_link"/>
+    <child link="left_finger_contact_link"/>
+    <origin xyz="-0.0265 0.012499 -0.19895" rpy="0 0 0"/>
+  </joint>
+  <joint name="right_finger_contact_joint" type="fixed">
+    <parent link="right_finger_tip_link"/>
+    <child link="right_finger_contact_link"/>
+    <origin xyz="0.0265 0.012499 -0.199024" rpy="0 0 0"/>
+  </joint>
   <link name="left_finger_inner_link">
     <!-- <inertial>
@@ -208,5 +220,5 @@
     <!-- <limit upper="0.523599" lower="-0.610865" effort="100" velocity="1.0"/> -->
   </joint>
-  <joint name="right_finger_outer_joint" type="fixed">
+  <joint name="right_finger_outer_joint" type="revolute">
     <origin xyz="0.0081 0.0128 0.085" rpy="0 0 0"/>
     <parent link="gripper_body_link"/>
@@ -215,7 +227,7 @@
     <dynamics damping="0.1"/>
     <limit upper="0.610865" lower="-0.610865" effort="100" velocity="1.0"/>
-    <!-- <mimic joint="left_finger_outer_joint" multiplier="-1"/> -->
-  </joint>
-  <joint name="left_finger_tip_joint" type="fixed">
+    <mimic joint="left_finger_outer_joint" multiplier="-1"/>
+  </joint>
+  <joint name="left_finger_tip_joint" type="revolute">
     <origin xyz="0.047384 -0.0253 0.06442" rpy="0 0 0"/>
     <parent link="left_finger_outer_link"/>
@@ -224,7 +236,7 @@
     <dynamics damping="0.1"/>
     <limit upper="0.610865" lower="-0.610865" effort="100" velocity="1.0"/>
-    <!-- <mimic joint="left_finger_outer_joint" multiplier="1"/> -->
-  </joint>
-  <joint name="right_finger_tip_joint" type="fixed">
+    <mimic joint="left_finger_outer_joint" multiplier="1"/>
+  </joint>
+  <joint name="right_finger_tip_joint" type="revolute">
     <origin xyz="-0.047384 -0.0253 0.064494" rpy="0 0 0"/>
     <parent link="right_finger_outer_link"/>
@@ -233,7 +245,7 @@
     <dynamics damping="0.1"/>
     <limit upper="0.610865" lower="-0.610865" effort="100" velocity="1.0"/>
-    <!-- <mimic joint="left_finger_outer_joint" multiplier="-1"/> -->
-  </joint>
-  <joint name="left_finger_inner_joint" type="fixed">
+    <mimic joint="left_finger_outer_joint" multiplier="-1"/>
+  </joint>
+  <joint name="left_finger_inner_joint" type="revolute">
     <origin xyz="0.0424 0.0001 0.1081" rpy="0 0 0"/>
     <parent link="gripper_body_link"/>
@@ -242,7 +254,7 @@
     <dynamics damping="0.1"/>
     <limit upper="0.610865" lower="-0.610865" effort="100" velocity="1.0"/>
-    <!-- <mimic joint="left_finger_outer_joint" multiplier="-1"/> -->
-  </joint>
-  <joint name="right_finger_inner_joint" type="fixed">
+    <mimic joint="left_finger_outer_joint" multiplier="-1"/>
+  </joint>
+  <joint name="right_finger_inner_joint" type="revolute">
     <origin xyz="0.0214 0.0001 0.1081" rpy="0 0 0"/>
     <parent link="gripper_body_link"/>
@@ -251,5 +263,5 @@
     <dynamics damping="0.1"/>
     <limit upper="0.610865" lower="-0.610865" effort="100" velocity="1.0"/>
-    <!-- <mimic joint="left_finger_outer_joint" multiplier="-1"/> -->
+    <mimic joint="left_finger_outer_joint" multiplier="-1"/>
   </joint>
   <joint name="tool0_joint" type="fixed">

File: my_robot_description/urdf/my_robot.ros2_control.xacro (robot description, xacro)
@@ -55,4 +55,19 @@
       <state_interface name="velocity"/>
     </joint>
+    <joint name="right_finger_outer_joint">
+      <state_interface name="position"/>
+    </joint>
+    <joint name="left_finger_tip_joint">
+      <state_interface name="position"/>
+    </joint>
+    <joint name="right_finger_tip_joint">
+      <state_interface name="position"/>
+    </joint>
+    <joint name="left_finger_inner_joint">
+      <state_interface name="position"/>
+    </joint>
+    <joint name="right_finger_inner_joint">
+      <state_interface name="position"/>
+    </joint>
   </ros2_control>
 </robot>
